Commit message: sdf

File: file1.urdf (robot description, URDF)
Before this commit: robot origins, 7 links, 6 joints
Joints:
- joint link1_link2: limit lower=-1 upper=0.785 effort=1000.0 velocity=0.5 -> lower=-2.57 upper=2.5 effort=1000.0 velocity=0.5
- joint link2_link3: limit lower=-0.785 upper=0.785 effort=1000.0 velocity=0.5 -> lower=-2.0 upper=2.0 effort=1000.0 velocity=0.5
