Commit message: calibrate directions

File: file-with-tool.urdf (robot description, URDF)
Before this commit: robot origins, 8 links, 7 joints
Joints:
- joint link6_link7: origin xyz=0.055 0 0.0025 rpy=0 -1.57 0 -> xyz=0.055 0 0.0025 rpy=-1.57 3.14 0

Commit message: with bounds and orientation

File: file-with-tool.urdf (robot description, URDF)
Before this commit: robot origins, 8 links, 7 joints
Joints:
- joint base_link_link1: limit lower=-1.57 upper=1.57 effort=1000.0 velocity=0.5 -> lower=-1.55 upper=1.35 effort=1000.0 velocity=0.5
- joint link1_link2: limit lower=-2.57 upper=2.5 effort=1000.0 velocity=0.5 -> lower=-1.2 upper=1 effort=1000.0 velocity=0.5
- joint link2_link3: limit lower=-2.0 upper=2.0 effort=1000.0 velocity=0.5 -> lower=-2.0 upper=1.2 effort=1000.0 velocity=0.5
- joint link3_link4: limit lower=-1.57 upper=1.57 effort=1000.0 velocity=0.5 -> lower=-0.55 upper=2.75 effort=1000.0 velocity=0.5
- joint link4_link5: limit lower=-1.57 upper=1.57 effort=1000.0 velocity=0.5 -> lower=-1.2 upper=0.55 effort=1000.0 velocity=0.5
- joint link5_link6: limit lower=1.57 upper=-1.57 effort=1000.0 velocity=0.5 -> lower=-1.55 upper=1.9 effort=1000.0 velocity=0.5
