Commit message: kalibration

File: file-with-tool2.urdf (robot description, URDF)
Before this commit: robot origins, 8 links, 7 joints
Joints:
- joint link1_link2: origin xyz=0 0.033 0.095 rpy=0 1.57 0 -> xyz=0 0.033 0.095 rpy=0 1.570796 0
- joint link3_link4: origin xyz=-0.02 0 0 rpy=-1.57 0 0 -> xyz=-0.02 0 0 rpy=-1.570796 0 0
- joint link4_link5: origin xyz=0 0 0.133 rpy=1.57 0 0 -> xyz=0 0 0.133 rpy=1.570796 0 0
- joint link5_link6: origin xyz=0 0.03 0 rpy=-1.57 0 0 -> xyz=0 0.03 0 rpy=-1.570796 0 0
- joint link6_link7: origin xyz=0.01 0.01 0.03 rpy=0 -1.57 0.785 -> xyz=0.01 0.01 0.03 rpy=0 -1.570796 1.0
